Commit message: Added upper_base_link to grasshopper, and modified base_link_to_laser joint accordingly, also changed the color of base link.

File: urdf/grass_hopper.urdf.xacro (robot description, xacro)
@@ -61,6 +61,6 @@
     <visual>
       <material>
-        <ambient>0.8392 0.6314 0.0 1.0</ambient>
-        <diffuse>0.8392 0.6314 0.0 1.0</diffuse>
+        <ambient>0.4 0.4 0.4 1.0</ambient>
+        <diffuse>0.4 0.4 0.4 1.0</diffuse>
         <specular>0.99 0.99 0.99 1.0</specular>
         <emissive>0.0 0.0 0.0 0.0</emissive>
@@ -68,4 +68,39 @@
     </visual>
   </gazebo>
+  <link name="upper_base_link">
+    <visual>
+      <origin xyz="-0.3 -0.1325 0" rpy="1.57 0 1.57" />
+      <geometry>
+        <mesh filename="file:///home/dhaval_lad/dhaval_ws/src/grasshopper_description/meshes/upper_base_link.stl" scale="0.001 0.001 0.001" />
+      </geometry>
+      <material name="grey"/>
+    </visual>
+    <collision>
+      <origin xyz="-0.3 -0.1325 0" rpy="1.57 0 1.57" />
+      <geometry>
+        <mesh filename="file:///home/dhaval_lad/dhaval_ws/src/grasshopper_description/meshes/upper_base_link.stl" scale="0.001 0.001 0.001" />
+      </geometry>
+    </collision>
+    <inertial>
+      <origin xyz="0 0 0" rpy="0 0 0" />
+      <mass value="1" />
+      <inertia ixx="8.438416e-3" ixy="0" ixz="0" iyy="0.0324083" iyz="0" izz="0.03603008" />
+    </inertial>
+  </link>
+  <gazebo reference="upper_base_link">
+    <visual>
+      <material>
+        <ambient>0.75 0.75 0.75 1.0</ambient>
+        <diffuse>0.75 0.75 0.75 1.0</diffuse>
+        <specular>0.99 0.99 0.99 1.0</specular>
+        <emissive>0.0 0.0 0.0 0.0</emissive>
+      </material>
+    </visual>
+  </gazebo>
+  <joint name="base_link_to_upper_base_link" type="fixed">
+    <parent link="base_link" />
+    <child link="upper_base_link" />
+    <origin xyz="0 0 0.165"/>
+  </joint>
   <link name="left_front_wheel">
     <visual>
@@ -285,5 +320,6 @@
     <parent link="base_link"/>
     <child link="laser"/>
-    <origin xyz="0.263 0 0.215" rpy="0 0 0" />
+    <!-- <origin xyz="0.263 0 0.245" rpy="0 0 0" />  -->   <!-- without upper base -->
+    <origin xyz="0 0 0.48" rpy="0 0 0" />   <!-- with upper base -->
   </joint>
   <gazebo reference="laser">
